Commit message: add initial four wheel drive

File: mammoth_description/urdf/mammoth.urdf (robot description, URDF)
Before this commit: robot mammoth, 5 links, 4 joints
Links:
- removed link caster_front
- added link wheel_fl, mass 1.1; collision cylinder length=0.075 radius=0.125; visual cylinder length=0.075 radius=0.125
- added link wheel_fr, mass 1.1; collision cylinder length=0.075 radius=0.125; visual cylinder length=0.075 radius=0.125
Joints:
- removed joint base_to_caster_front
- added joint base_to_wheel_fl: type continuous, parent base_link, child wheel_fl, origin xyz=-0.3 -0.2375 -0.1 rpy=1.57 -3.14159 0, axis 0 0 1
- added joint base_to_wheel_fr: type continuous, parent base_link, child wheel_fr, origin xyz=-0.3 0.2375 -0.1 rpy=1.57 -3.14159 0, axis 0 0 1

Commit message: add rudimentary treads

File: mammoth_description/urdf/mammoth.urdf (robot description, URDF)
Before this commit: robot mammoth, 7 links, 6 joints
Links:
- added link wheel_al, mass 1.1; collision cylinder length=0.075 radius=0.125; visual cylinder length=0.075 radius=0.125
- added link wheel_ar, mass 1.1; collision cylinder length=0.075 radius=0.125; visual cylinder length=0.075 radius=0.125
- added link wheel_ml, mass 1.1; collision cylinder length=0.075 radius=0.125; visual cylinder length=0.075 radius=0.125
- added link wheel_mr, mass 1.1; collision cylinder length=0.075 radius=0.125; visual cylinder length=0.075 radius=0.125
- added link wheel_pl, mass 1.1; collision cylinder length=0.075 radius=0.125; visual cylinder length=0.075 radius=0.125
- added link wheel_pr, mass 1.1; collision cylinder length=0.075 radius=0.125; visual cylinder length=0.075 radius=0.125
Joints:
- added joint base_to_wheel_al: type continuous, parent base_link, child wheel_al, origin xyz=0.15 -0.2375 -0.1 rpy=1.57 -3.14159 0, axis 0 0 1
- added joint base_to_wheel_ar: type continuous, parent base_link, child wheel_ar, origin xyz=0.15 0.2375 -0.1 rpy=1.57 -3.14159 0, axis 0 0 1
- added joint base_to_wheel_ml: type continuous, parent base_link, child wheel_ml, origin xyz=0 -0.2375 -0.1 rpy=1.57 -3.14159 0, axis 0 0 1
- added joint base_to_wheel_mr: type continuous, parent base_link, child wheel_mr, origin xyz=0 0.2375 -0.1 rpy=1.57 -3.14159 0, axis 0 0 1
- added joint base_to_wheel_pl: type continuous, parent base_link, child wheel_pl, origin xyz=-0.15 -0.2375 -0.1 rpy=1.57 -3.14159 0, axis 0 0 1
- added joint base_to_wheel_pr: type continuous, parent base_link, child wheel_pr, origin xyz=-0.15 0.2375 -0.1 rpy=1.57 -3.14159 0, axis 0 0 1

Commit message: fix urdf so that pointclouds are published, add base_footprint, clean up ros_ign_bridge launch

File: mammoth_description/urdf/mammoth.urdf (robot description, URDF)
Before this commit: robot mammoth, 6 links, 5 joints
Links:
- added link base_footprint
Joints:
- added joint base_footprint_to_base_link: type fixed, parent base_footprint, child base_link, origin xyz=0 0 0.225 rpy=0 0 0

Commit message: fix publishing rate issue

File: mammoth_description/urdf/mammoth.urdf (robot description, URDF)
Before this commit: robot mammoth, 13 links, 12 joints
Links:
- link base_link: mass None -> 45

Commit message: slam changes

File: mammoth_description/urdf/mammoth.urdf (robot description, URDF)
Before this commit: robot mammoth, 13 links, 12 joints
Links:
- added link imu_link, mass 1e-5; collision cylinder length=0.05 radius=0.025; visual cylinder length=0.05 radius=0.025
Joints:
- added joint base_to_imu: type fixed, parent base_link, child imu_link, origin xyz=0 0 0.175 rpy=0 0 0

Commit message: slam up and running

File: mammoth_description/urdf/mammoth.urdf (robot description, URDF)
Before this commit: robot mammoth, 14 links, 13 joints
Links:
- link base_link: mass 45 -> None

Commit message: orientation of wheels fixed

File: mammoth_description/urdf/mammoth.urdf (robot description, URDF)
Before this commit: robot mammoth, 14 links, 13 joints
Joints:
- joint base_to_wheel_al: origin xyz=0.15 -0.2375 -0.1 rpy=1.57 -3.14159 0 -> xyz=0.15 -0.2375 -0.1 rpy=1.57 -3.14159 -3.14159
- joint base_to_wheel_ar: origin xyz=0.15 0.2375 -0.1 rpy=1.57 -3.14159 0 -> xyz=0.15 0.2375 -0.1 rpy=1.57 -3.14159 -3.14159
- joint base_to_wheel_bl: origin xyz=0.3 -0.2375 -0.1 rpy=1.57 -3.14159 0 -> xyz=0.3 -0.2375 -0.1 rpy=1.57 -3.14159 -3.14159
- joint base_to_wheel_br: origin xyz=0.3 0.2375 -0.1 rpy=1.57 -3.14159 0 -> xyz=0.3 0.2375 -0.1 rpy=1.57 -3.14159 -3.14159
- joint base_to_wheel_fl: origin xyz=-0.3 -0.2375 -0.1 rpy=1.57 -3.14159 0 -> xyz=-0.3 -0.2375 -0.1 rpy=1.57 -3.14159 -3.14159
- joint base_to_wheel_fr: origin xyz=-0.3 0.2375 -0.1 rpy=1.57 -3.14159 0 -> xyz=-0.3 0.2375 -0.1 rpy=1.57 -3.14159 -3.14159
- joint base_to_wheel_ml: origin xyz=0 -0.2375 -0.1 rpy=1.57 -3.14159 0 -> xyz=0 -0.2375 -0.1 rpy=1.57 -3.14159 -3.14159
- joint base_to_wheel_mr: origin xyz=0 0.2375 -0.1 rpy=1.57 -3.14159 0 -> xyz=0 0.2375 -0.1 rpy=1.57 -3.14159 -3.14159
- joint base_to_wheel_pl: origin xyz=-0.15 -0.2375 -0.1 rpy=1.57 -3.14159 0 -> xyz=-0.15 -0.2375 -0.1 rpy=1.57 -3.14159 -3.14159
- joint base_to_wheel_pr: origin xyz=-0.15 0.2375 -0.1 rpy=1.57 -3.14159 0 -> xyz=-0.15 0.2375 -0.1 rpy=1.57 -3.14159 -3.14159

File: mammoth_description/urdf/mammoth1.urdf (robot description, URDF)
Before this commit: robot mammoth, 14 links, 13 joints
Joints:
- joint base_to_imu: origin xyz=0 0 0.175 rpy=0 0 0 -> xyz=0.3048 0 0.175 rpy=0 0 0
- joint base_to_laser: origin xyz=0 0 0.175 rpy=0 0 0 -> xyz=0.3048 0 0.175 rpy=0 0 0
- joint base_to_wheel_al: origin xyz=0.15 -0.2375 -0.1 rpy=1.57 -3.14159 0 -> xyz=0.15 0.2375 -0.1 rpy=1.57 -3.14159 -3.14159; type fixed -> continuous
- joint base_to_wheel_ar: origin xyz=0.15 0.2375 -0.1 rpy=1.57 -3.14159 0 -> xyz=0.15 -0.2375 -0.1 rpy=1.57 -3.14159 -3.14159; type fixed -> continuous
- joint base_to_wheel_bl: origin xyz=0.3 -0.2375 -0.1 rpy=1.57 -3.14159 0 -> xyz=0.3 0.2375 -0.1 rpy=1.57 -3.14159 -3.14159; type fixed -> continuous
- joint base_to_wheel_br: origin xyz=0.3 0.2375 -0.1 rpy=1.57 -3.14159 0 -> xyz=0.3 -0.2375 -0.1 rpy=1.57 -3.14159 -3.14159; type fixed -> continuous
- joint base_to_wheel_fl: origin xyz=-0.3 -0.2375 -0.1 rpy=1.57 -3.14159 0 -> xyz=-0.3 0.2375 -0.1 rpy=1.57 -3.14159 -3.14159; type fixed -> continuous
- joint base_to_wheel_fr: origin xyz=-0.3 0.2375 -0.1 rpy=1.57 -3.14159 0 -> xyz=-0.3 -0.2375 -0.1 rpy=1.57 -3.14159 -3.14159; type fixed -> continuous
- joint base_to_wheel_ml: origin xyz=0 -0.2375 -0.1 rpy=1.57 -3.14159 0 -> xyz=0 0.2375 -0.1 rpy=1.57 -3.14159 -3.14159; type fixed -> continuous
- joint base_to_wheel_mr: origin xyz=0 0.2375 -0.1 rpy=1.57 -3.14159 0 -> xyz=0 -0.2375 -0.1 rpy=1.57 -3.14159 -3.14159; type fixed -> continuous
- joint base_to_wheel_pl: origin xyz=-0.15 -0.2375 -0.1 rpy=1.57 -3.14159 0 -> xyz=-0.15 0.2375 -0.1 rpy=1.57 -3.14159 -3.14159; type fixed -> continuous
- joint base_to_wheel_pr: origin xyz=-0.15 0.2375 -0.1 rpy=1.57 -3.14159 0 -> xyz=-0.15 -0.2375 -0.1 rpy=1.57 -3.14159 -3.14159; type fixed -> continuous

Commit message: base_footprint, and lidar/imu movement

File: mammoth_description/urdf/mammoth.urdf (robot description, URDF)
Before this commit: robot mammoth, 14 links, 13 joints
Joints:
- joint base_footprint_to_base_link: origin xyz=0 0 0.225 rpy=0 0 0 -> xyz=0 0 0.225 rpy=0 0 3.14
- joint base_to_imu: origin xyz=0 0 0.175 rpy=0 0 0 -> xyz=-0.3048 0 0.175 rpy=0 0 3.14
- joint base_to_laser: origin xyz=0 0 0.175 rpy=0 0 0 -> xyz=-0.3048 0 0.175 rpy=0 0 3.14
- joint base_to_wheel_al: origin xyz=0.15 -0.2375 -0.1 rpy=1.57 -3.14159 -3.14159 -> xyz=0.15 -0.2375 -0.1 rpy=1.57 -3.14159 0
- joint base_to_wheel_ar: origin xyz=0.15 0.2375 -0.1 rpy=1.57 -3.14159 -3.14159 -> xyz=0.15 0.2375 -0.1 rpy=1.57 -3.14159 0
- joint base_to_wheel_bl: origin xyz=0.3 -0.2375 -0.1 rpy=1.57 -3.14159 -3.14159 -> xyz=0.3 -0.2375 -0.1 rpy=1.57 -3.14159 0
- joint base_to_wheel_br: origin xyz=0.3 0.2375 -0.1 rpy=1.57 -3.14159 -3.14159 -> xyz=0.3 0.2375 -0.1 rpy=1.57 -3.14159 0
- joint base_to_wheel_fl: origin xyz=-0.3 -0.2375 -0.1 rpy=1.57 -3.14159 -3.14159 -> xyz=-0.3 -0.2375 -0.1 rpy=1.57 -3.14159 0
- joint base_to_wheel_fr: origin xyz=-0.3 0.2375 -0.1 rpy=1.57 -3.14159 -3.14159 -> xyz=-0.3 0.2375 -0.1 rpy=1.57 -3.14159 0
- joint base_to_wheel_ml: origin xyz=0 -0.2375 -0.1 rpy=1.57 -3.14159 -3.14159 -> xyz=0 -0.2375 -0.1 rpy=1.57 -3.14159 0
- joint base_to_wheel_mr: origin xyz=0 0.2375 -0.1 rpy=1.57 -3.14159 -3.14159 -> xyz=0 0.2375 -0.1 rpy=1.57 -3.14159 0
- joint base_to_wheel_pl: origin xyz=-0.15 -0.2375 -0.1 rpy=1.57 -3.14159 -3.14159 -> xyz=-0.15 -0.2375 -0.1 rpy=1.57 -3.14159 0
- joint base_to_wheel_pr: origin xyz=-0.15 0.2375 -0.1 rpy=1.57 -3.14159 -3.14159 -> xyz=-0.15 0.2375 -0.1 rpy=1.57 -3.14159 0

File: mammoth_description/urdf/mammoth1.urdf (robot description, URDF)
Before this commit: robot mammoth, 14 links, 13 joints
Joints:
- joint base_footprint_to_base_link: origin xyz=0 0 0.225 rpy=0 0 0 -> xyz=0 0 0.225 rpy=0 0 3.14
- joint base_to_imu: origin xyz=0.3048 0 0.175 rpy=0 0 0 -> xyz=-0.3048 0 0.175 rpy=0 0 3.14
- joint base_to_laser: origin xyz=0.3048 0 0.175 rpy=0 0 0 -> xyz=-0.3048 0 0.175 rpy=0 0 3.14
- joint base_to_wheel_al: origin xyz=0.15 0.2375 -0.1 rpy=1.57 -3.14159 -3.14159 -> xyz=0.15 -0.2375 -0.1 rpy=1.57 -3.14159 0
- joint base_to_wheel_ar: origin xyz=0.15 -0.2375 -0.1 rpy=1.57 -3.14159 -3.14159 -> xyz=0.15 0.2375 -0.1 rpy=1.57 -3.14159 0
- joint base_to_wheel_bl: origin xyz=0.3 0.2375 -0.1 rpy=1.57 -3.14159 -3.14159 -> xyz=0.3 -0.2375 -0.1 rpy=1.57 -3.14159 0
- joint base_to_wheel_br: origin xyz=0.3 -0.2375 -0.1 rpy=1.57 -3.14159 -3.14159 -> xyz=0.3 0.2375 -0.1 rpy=1.57 -3.14159 0
- joint base_to_wheel_fl: origin xyz=-0.3 0.2375 -0.1 rpy=1.57 -3.14159 -3.14159 -> xyz=-0.3 -0.2375 -0.1 rpy=1.57 -3.14159 0
- joint base_to_wheel_fr: origin xyz=-0.3 -0.2375 -0.1 rpy=1.57 -3.14159 -3.14159 -> xyz=-0.3 0.2375 -0.1 rpy=1.57 -3.14159 0
- joint base_to_wheel_ml: origin xyz=0 0.2375 -0.1 rpy=1.57 -3.14159 -3.14159 -> xyz=0 -0.2375 -0.1 rpy=1.57 -3.14159 0
- joint base_to_wheel_mr: origin xyz=0 -0.2375 -0.1 rpy=1.57 -3.14159 -3.14159 -> xyz=0 0.2375 -0.1 rpy=1.57 -3.14159 0
- joint base_to_wheel_pl: origin xyz=-0.15 0.2375 -0.1 rpy=1.57 -3.14159 -3.14159 -> xyz=-0.15 -0.2375 -0.1 rpy=1.57 -3.14159 0
- joint base_to_wheel_pr: origin xyz=-0.15 -0.2375 -0.1 rpy=1.57 -3.14159 -3.14159 -> xyz=-0.15 0.2375 -0.1 rpy=1.57 -3.14159 0

Commit message: Ros2 urdf fix (#60)

File: mammoth_description/urdf/mammoth.urdf (robot description, URDF)
Before this commit: robot mammoth, 14 links, 13 joints
Joints:
- joint base_footprint_to_base_link: origin xyz=0 0 0.225 rpy=0 0 0 -> xyz=0 0 0.225 rpy=0 0 3.14
- joint base_to_imu: origin xyz=0 0 0.175 rpy=0 0 0 -> xyz=-0.3048 0 0.175 rpy=0 0 3.14
- joint base_to_laser: origin xyz=0 0 0.175 rpy=0 0 0 -> xyz=-0.3048 0 0.175 rpy=0 0 3.14

File: mammoth_description/urdf/mammoth1.urdf (robot description, URDF)
Before this commit: robot mammoth, 14 links, 13 joints
Joints:
- joint base_footprint_to_base_link: origin xyz=0 0 0.225 rpy=0 0 0 -> xyz=0 0 0.225 rpy=0 0 3.14
- joint base_to_imu: origin xyz=0 0 0.175 rpy=0 0 0 -> xyz=-0.3048 0 0.175 rpy=0 0 3.14
- joint base_to_laser: origin xyz=0 0 0.175 rpy=0 0 0 -> xyz=-0.3048 0 0.175 rpy=0 0 3.14
- joint base_to_wheel_al: type fixed -> continuous
- joint base_to_wheel_ar: type fixed -> continuous
- joint base_to_wheel_bl: type fixed -> continuous
- joint base_to_wheel_br: type fixed -> continuous
- joint base_to_wheel_fl: type fixed -> continuous
- joint base_to_wheel_fr: type fixed -> continuous
- joint base_to_wheel_ml: type fixed -> continuous
- joint base_to_wheel_mr: type fixed -> continuous
- joint base_to_wheel_pl: type fixed -> continuous
- joint base_to_wheel_pr: type fixed -> continuous
