Commit message: gazebo update

File: mammoth_description/urdf/mammoth1.urdf (robot description, URDF)
Before this commit: robot mammoth, 19 links, 18 joints
Links:
- removed link zed_camera_center
- removed link zed_left_camera_frame
- removed link zed_left_camera_optical_frame
- removed link zed_right_camera_frame
- removed link zed_right_camera_optical_frame
Joints:
- removed joint zed_camera_center_joint
- removed joint zed_left_camera_joint
- removed joint zed_left_camera_optical_joint
- removed joint zed_right_camera_joint
- removed joint zed_right_camera_optical_joint

Commit message: lidar and imu orientation fix

File: mammoth_description/urdf/mammoth1.urdf (robot description, URDF)
Before this commit: robot mammoth, 14 links, 13 joints
Joints:
- joint base_to_imu: origin xyz=-0.3048 0 0.175 rpy=0 0 3.14 -> xyz=-0.3048 0 0.175 rpy=0 0 0
- joint base_to_laser: origin xyz=-0.3048 0 0.175 rpy=0 0 3.14 -> xyz=-0.3048 0 0.175 rpy=0 0 0
